File: Half Bridge - 6S 50A.kicad_sch (KiCad schematic)
At the start: 6 parts

Commit message: Fixed pin names
reset pins to apply proper net names
Parts:
- renumbered A1 to B1
Changed lines of the file:
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@@
 		(dnp no)
 		(fields_autoplaced yes)
-		(property "Reference" "A1"
+		(property "Reference" "B1"
 			(at 116.84 102.8699 90)
 			(effects

Commit message: more routing
Parts:
- renumbered B1 to A1, B_High1 to A_High1, B_Low1 to A_Low1, R_Gate_B_High1 to R_Gate_A_High1, R_Gate_B_Low1 to R_Gate_A_Low1
Connections:
- net X: now reaches A1.1, A_High1.1 (SOURCE), A_High1.2 (SOURCE), A_High1.3 (SOURCE), A_Low1.5 (DRAIN), A_Low1.6 (DRAIN), A_Low1.7 (DRAIN), A_Low1.8 (DRAIN), C13.2
- net -BATT: now reaches A_Low1.1 (SOURCE), A_Low1.2 (SOURCE), A_Low1.3 (SOURCE)
- net +BATT: now reaches A_High1.5 (DRAIN), A_High1.6 (DRAIN), A_High1.7 (DRAIN), A_High1.8 (DRAIN)
Other:
- moved on the sheet: A1

Commit message: more routing and placement
Parts:
- renumbered A1 to A4, C13 to C26
Connections:
- net +BATT: no longer A_High1.6 (DRAIN), A_High1.7 (DRAIN), A_High1.8 (DRAIN)
- net X: no longer A_Low1.6 (DRAIN), A_Low1.7 (DRAIN), A_Low1.8 (DRAIN)
Other:
- moved on the sheet: A_High1, A_Low1
