File: MCU.kicad_sch (KiCad schematic)
At the start: 5 parts, among them U8 STM32G071GBU3TR

Commit message: Fixed pin names
reset pins to apply proper net names
Parts:
- removed R21: 1K, Resistor_SMD:R_0402_1005Metric, symbol Device:R_US
- added R14: 1K, Resistor_SMD:R_0402_1005Metric, symbol Device:R_US
- U8: footprint STM32:UFQFPN-28 -> STM32 G0:UFQFPN-28
Connections:
- net DShot: now also R14.2
- net DShotTXRX: now reaches U8.24 (PB4), U8.25 (PB5)
- net DShotTXRX: now also R14.1
Changed lines of the file:
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@@
+	(wire
+		(pts
+			(xy 255.27 88.9) (xy 251.46 88.9)
+		)
+		(stroke
+			(width 0)
+			(type default)
+		)
+	)
 	(wire
 		(pts
@@
 	(wire
 		(pts
+			(xy 237.49 88.9) (xy 243.84 88.9)
+		)
+		(stroke
+			(width 0)
+			(type default)
+		)
+	)
+	(wire
+		(pts
 			(xy 186.69 96.52) (xy 176.53 96.52)
 		)
@@
 	(wire
 		(pts
-			(xy 209.55 90.17) (xy 203.2 90.17)
-		)
-		(stroke
-			(width 0)
-			(type default)
-		)
-	)
-	(wire
-		(pts
 			(xy 179.07 90.17) (xy 179.07 88.9)
 		)
@@
 		)
 	)
+	(label "DShotTXRX"
+		(at 255.27 88.9 0)
+		(effects
+			(font
+				(size 1.27 1.27)
+			)
+			(justify left bottom)
+		)
+	)
+	(label "DShotTXRX"
+		(at 195.58 90.17 0)
+		(effects
+			(font
+				(size 1.27 1.27)
+			)
+			(justify left bottom)
+		)
+	)
+	(hierarchical_label "SWD_CLK"
+		(shape input)
+		(at 80.01 111.76 180)
+		(effects
+			(font
+				(size 1.27 1.27)
+			)
+			(justify right)
+		)
+	)
+	(hierarchical_label "Batt_Sense"
+		(shape input)
+		(at 95.25 83.82 180)
+		(effects
+			(font
+				(size 1.27 1.27)
+			)
+			(justify right)
+		)
+	)
+	(hierarchical_label "PWM_H_A"
+		(shape input)
+		(at 95.25 106.68 180)
+		(effects
+			(font
+				(size 1.27 1.27)
+			)
+			(justify right)
+		)
+	)
+	(hierarchical_label "ZC_C"
+		(shape input)
+		(at 95.25 86.36 180)
+		(effects
+			(font
+				(size 1.27 1.27)
+			)
+			(justify right)
+		)
+	)
+	(hierarchical_label "PWM_L_B"
+		(shape input)
+		(at 182.88 81.28 0)
+		(effects
+			(font
+				(size 1.27 1.27)
+			)
+			(justify left)
+		)
+	)
 	(hierarchical_label "DShot"
 		(shape input)
-		(at 209.55 90.17 0)
-		(effects
-			(font
-				(size 1.27 1.27)
-			)
-			(justify left)
-		)
-	)
-	(hierarchical_label "SWD_CLK"
-		(shape input)
-		(at 80.01 111.76 180)
+		(at 237.49 88.9 180)
 		(effects
 			(font
@@
 			)
 			(justify right)
-		)
-	)
-	(hierarchical_label "Batt_Sense"
-		(shape input)
-		(at 95.25 83.82 180)
-		(effects
-			(font
-				(size 1.27 1.27)
-			)
-			(justify right)
-		)
-	)
-	(hierarchical_label "PWM_H_A"
-		(shape input)
-		(at 95.25 106.68 180)
-		(effects
-			(font
-				(size 1.27 1.27)
-			)
-			(justify right)
-		)
-	)
-	(hierarchical_label "ZC_C"
-		(shape input)
-		(at 95.25 86.36 180)
-		(effects
-			(font
-				(size 1.27 1.27)
-			)
-			(justify right)
-		)
-	)
-	(hierarchical_label "PWM_L_B"
-		(shape input)
-		(at 182.88 81.28 0)
-		(effects
-			(font
-				(size 1.27 1.27)
-			)
-			(justify left)
 		)
 	)
@@
 			)
 		)
-		(property "Footprint" "STM32:UFQFPN-28"
+		(property "Footprint" "STM32 G0:UFQFPN-28"
 			(at 100.33 81.28 0)
 			(effects
@@
 			)
 		)
-		(property "Datasheet" "~"
+		(property "Datasheet" "https://mm.digikey.com/Volume0/opasdata/d220001/medias/docus/609/CL05B104KP5NNNC_Spec.pdf"
 			(at 179.07 121.92 0)
 			(effects
@@
 	(symbol
 		(lib_id "Device:R_US")
-		(at 199.39 90.17 90)
+		(at 247.65 88.9 270)
 		(unit 1)
 		(exclude_from_sim no)
@@
 		(on_board yes)
 		(dnp no)
-		(property "Reference" "R21"
-			(at 199.136 87.63 90)
+		(property "Reference" "R14"
+			(at 247.904 91.44 90)
 			(effects
 				(font
@@
 		)
 		(property "Value" "1K"
-			(at 199.644 92.71 90)
+			(at 248.666 86.36 90)
 			(effects
 				(font
@@
 		)
 		(property "Footprint" "Resistor_SMD:R_0402_1005Metric"
-			(at 199.644 89.154 90)
+			(at 247.396 89.916 90)
 			(effects
 				(font
@@
 		)
 		(property "Datasheet" "~"
-			(at 199.39 90.17 0)
+			(at 247.65 88.9 0)
 			(effects
 				(font
@@
 		)
 		(property "Description" "Resistor, US symbol"
-			(at 199.39 90.17 0)
+			(at 247.65 88.9 0)
 			(effects
 				(font
@@
 			(project "ESC"
 				(path "/0e826802-e676-4548-b85d-7973e5fc1500/dd4480c0-fc92-4865-b71a-49548ede0e1d/ce85d30a-5b72-4428-9ad8-811f15b427f8"
-					(reference "R21")
+					(reference "R14")
 					(unit 1)
 				)

Commit message: more routing and placement
Parts:
- renumbered C15 to C28, C16 to C29, R20 to R14, R14 to R15, U8 to U4
