File: Power Input.kicad_sch (KiCad schematic)
At the start: 29 parts, among them U10 AP7381-33SA-7, U9 UA78L10ACPK

Commit message: more routing
Connections:
- net +BATT: now also R1.1
- net -BATT: now also C28.2, C29.2, R2.2

Commit message: more routing and placement
Parts:
- renumbered C29 to C1, C4 to C10, C20 to C11, C5 to C12, C21 to C13, C6 to C14, C22 to C15, C7 to C16, C23 to C17, C8 to C18, C24 to C19, C27 to C2, C9 to C20, C25 to C21, C10 to C22, C26 to C23, C28 to C3, C1 to C4, C17 to C5, C2 to C6, C18 to C7, C3 to C8, C19 to C9, U9 to U1, U10 to U2
Connections:
- net +BATT: now also C10.1, C11.1, C12.1, C13.1, C14.1, C15.1, C16.1, C17.1, C18.1, C19.1, C20.1, C21.1, C22.1, C23.1, C4.1, C5.1, C6.1, C7.1, C8.1, C9.1
- net -BATT: now also C10.2, C11.2, C12.2, C13.2, C14.2, C15.2, C16.2, C17.2, C18.2, C19.2, C20.2, C21.2, C22.2, C23.2, C4.2, C5.2, C6.2, C7.2, C8.2, C9.2
